File: MEC1003F 2024 Lecture 3 Demo.kicad_sch (KiCad schematic)
At the start: 16 parts, among them U1 AP331AWRG-7, U2 AP331AWRG-7

Commit message: Apply Lecture 2 Changes Rename Project Update README.md
Parts:
- J1, J2: footprint (none) -> Project Footprints:CROC
- R1, R3, R4, R5, R6, R7, R8: footprint (none) -> Resistor_SMD:R_0603_1608Metric
- U1, U2: footprint (none) -> Project Footprints:SOT-23-5 (AP331A)
Changed lines of the file:
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@@
       (effects (font (size 1.27 1.27)))
     )
-    (property "Footprint" "" (at 200.66 142.24 90)
+    (property "Footprint" "Resistor_SMD:R_0603_1608Metric" (at 200.66 142.24 90)
       (effects (font (size 1.27 1.27)) hide)
     )
@@
       (effects (font (size 1.27 1.27)))
     )
-    (property "Footprint" "" (at 29.21 17.78 0)
+    (property "Footprint" "Project Footprints:CROC" (at 29.21 17.78 0)
       (effects (font (size 1.27 1.27)) hide)
     )
@@
       (effects (font (size 1.27 1.27)) (justify left))
     )
-    (property "Footprint" "" (at 71.12 123.19 90)
+    (property "Footprint" "Resistor_SMD:R_0603_1608Metric" (at 71.12 123.19 90)
       (effects (font (size 1.27 1.27)) hide)
     )
@@
       (effects (font (size 1.27 1.27)))
     )
-    (property "Footprint" "" (at 116.84 142.24 90)
+    (property "Footprint" "Resistor_SMD:R_0603_1608Metric" (at 116.84 142.24 90)
       (effects (font (size 1.27 1.27)) hide)
     )
@@
       (effects (font (size 1.27 1.27)))
     )
-    (property "Footprint" "" (at 29.21 43.18 0)
+    (property "Footprint" "Project Footprints:CROC" (at 29.21 43.18 0)
       (effects (font (size 1.27 1.27)) hide)
     )
@@
       (effects (font (size 1.27 1.27)) (justify left))
     )
-    (property "Footprint" "" (at 165.1 146.05 90)
+    (property "Footprint" "Resistor_SMD:R_0603_1608Metric" (at 165.1 146.05 90)
       (effects (font (size 1.27 1.27)) hide)
     )
@@
       (effects (font (size 1.27 1.27)) (justify left))
     )
-    (property "Footprint" "" (at 165.1 123.19 90)
+    (property "Footprint" "Resistor_SMD:R_0603_1608Metric" (at 165.1 123.19 90)
       (effects (font (size 1.27 1.27)) hide)
     )
@@
       (effects (font (size 1.27 1.27)))
     )
-    (property "Footprint" "" (at 111.76 147.32 0)
+    (property "Footprint" "Project Footprints:SOT-23-5 (AP331A)" (at 111.76 147.32 0)
       (effects (font (size 1.27 1.27)) hide)
     )
@@
       (effects (font (size 1.27 1.27)) (justify left))
     )
-    (property "Footprint" "" (at 139.7 105.41 90)
+    (property "Footprint" "Resistor_SMD:R_0603_1608Metric" (at 139.7 105.41 90)
       (effects (font (size 1.27 1.27)) hide)
     )
@@
       (effects (font (size 1.27 1.27)) (justify left))
     )
-    (property "Footprint" "" (at 71.12 146.05 90)
+    (property "Footprint" "Resistor_SMD:R_0603_1608Metric" (at 71.12 146.05 90)
       (effects (font (size 1.27 1.27)) hide)
     )
@@
       (effects (font (size 1.27 1.27)))
     )
-    (property "Footprint" "" (at 193.04 147.32 0)
-      (effects (font (size 1.27 1.27)) hide)
-    )
+    (property "Footprint" "Project Footprints:SOT-23-5 (AP331A)" (at 193.04 147.32 0)
+      (effects (font (size 1.27 1.27)) hide)
+    )
